File: Interuppter/charge.kicad_sch (KiCad schematic)
At the start: 28 parts, among them J2 Conn_01x03, J4 USB_C_Receptacle_USB2.0_16P, U6 IP2326, U7 USBLC6-2SC6

Commit message: Update KiCAD and add GERBER files and 3D screenshots
Parts:
- J2: footprint Conn_JST:JST_GH_SM03B-GHS-TB_1x03-1MP_P1.25mm_Horizontal -> Connector_Molex:Molex_PicoBlade_53261-0371_1x03-1MP_P1.25mm_Horizontal
Changed lines of the file:
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@@
 			)
 		)
-		(property "Footprint" "Conn_JST:JST_GH_SM03B-GHS-TB_1x03-1MP_P1.25mm_Horizontal"
+		(property "Footprint" "Connector_Molex:Molex_PicoBlade_53261-0371_1x03-1MP_P1.25mm_Horizontal"
 			(at 83.82 31.75 0)
 			(hide yes)
