File: Interuppter/Interuppter.kicad_sch (KiCad schematic)
At the start: 14 parts, among them J5 Display, SW2 BUT_START, U2 DRL2180_OUT, U5 DRL2180_IN

Commit message: Update C++ code
Other:
- note removed: "My display has a reversible connector. So, the connector itself is upside down."
Changed lines of the file:
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@@
-		)
-	)
-	(text "My display has a reversible connector. \nSo, the connector itself is upside down.\n"
-		(exclude_from_sim no)
-		(at 36.83 148.082 0)
-		(effects
-			(font
-				(size 1.27 1.27)
-			)
 		)
 	)
